Commit message: Keypoints Map2d Local Fix

File: Xarm7/assets/xarm7_gripper_origin/xarm7_with_gripper.urdf (robot description, URDF)
Before this commit: robot UF_ROBOT, 18 links, 17 joints
Joints:
- joint drive_joint: limit lower=0 upper=0.85 effort=50 velocity=2 -> lower=0 upper=0.85 effort=500 velocity=20
- joint joint1: limit lower=-6.283185307179586 upper=6.283185307179586 effort=50 velocity=3.14 -> lower=-6.283185307179586 upper=6.283185307179586 effort=500 velocity=31.4
- joint joint2: limit lower=-2.059 upper=2.0944 effort=50 velocity=3.14 -> lower=-2.059 upper=2.0944 effort=500 velocity=31.4
- joint joint3: limit lower=-6.283185307179586 upper=6.283185307179586 effort=30 velocity=3.14 -> lower=-6.283185307179586 upper=6.283185307179586 effort=300 velocity=31.4
- joint joint4: limit lower=-0.19198 upper=3.927 effort=30 velocity=3.14 -> lower=-0.19198 upper=3.927 effort=300 velocity=31.4
- joint joint5: limit lower=-6.283185307179586 upper=6.283185307179586 effort=30 velocity=3.14 -> lower=-6.283185307179586 upper=6.283185307179586 effort=300 velocity=31.4
- joint joint6: limit lower=-1.69297 upper=3.141592653589793 effort=20 velocity=3.14 -> lower=-1.69297 upper=3.141592653589793 effort=200 velocity=31.4
- joint joint7: limit lower=-6.283185307179586 upper=6.283185307179586 effort=20 velocity=3.14 -> lower=-6.283185307179586 upper=6.283185307179586 effort=200 velocity=31.4
- joint left_finger_joint: limit lower=0 upper=0.85 effort=50 velocity=2 -> lower=0 upper=0.85 effort=500 velocity=20
- joint left_inner_knuckle_joint: limit lower=0 upper=0.85 effort=50 velocity=2 -> lower=0 upper=0.85 effort=500 velocity=20
- joint right_finger_joint: limit lower=0 upper=0.85 effort=50 velocity=2 -> lower=0 upper=0.85 effort=500 velocity=20
- joint right_inner_knuckle_joint: limit lower=0 upper=0.85 effort=50 velocity=2 -> lower=0 upper=0.85 effort=500 velocity=20
- joint right_outer_knuckle_joint: limit lower=0 upper=0.85 effort=50 velocity=2 -> lower=0 upper=0.85 effort=500 velocity=20
